File: IEEE_Drone_2026/IEE_Drone_2026.kicad_sch (KiCad schematic)
At the start: 32 parts, among them IC1 TPSM84209RKHT, IC2 TPSM84209RKHT, J1 ESC, J10 M2, J11 Conn_01x02_Socket, J2 M4 Mounting, J3 M4 Mounting, J4 M4 Mounting, J5 M4 Mounting, J6 Pixy2, J7 M2, J8 M2, J9 M2, Q1 2N2222, U1 MS560702BA03-50, U2 ATSAMD21G18A-A

Commit message: added new schematic items
Parts:
- removed A1: Adafruit_Feather_M0_RFM9x_LoRa_Radio, Module:Adafruit_Feather_M0_RFM, symbol MCU_Module:Adafruit_Feather_M0_RFM9x_LoRa_Radio
- removed IC2: TPSM84209RKHT, TPSM84209RKHT, symbol TPSM84209RKHT:TPSM84209RKHT
- removed R5: 10k, Resistor_SMD:R_0603_1608Metric_Pad0.98x0.95mm_HandSolder, symbol Device:R
- removed R6: 1.1k, Resistor_SMD:R_0603_1608Metric_Pad0.98x0.95mm_HandSolder, symbol Device:R
- removed U2: ATSAMD21G18A-A, Package_QFP:TQFP-48_7x7mm_P0.5mm, symbol MCU_Microchip_SAMD:ATSAMD21G18A-A
- added C8: 12pF, Capacitor_SMD:C_0603_1608Metric_Pad1.08x0.95mm_HandSolder, symbol Device:C
- added J12: RF, symbol Connector:Conn_01x09_Socket
- added J13: USB_C_Receptacle_USB2.0_16P, symbol Connector:USB_C_Receptacle_USB2.0_16P
- added MT1: ICM-42605, ICM-42605:XDCR_ICM-42605, symbol ICM-42605:ICM-42605
- added U2: STM32F405RGTx, Package_QFP:LQFP-64_10x10mm_P0.5mm, symbol MCU_ST_STM32F4:STM32F405RGTx
- added U3: BMP280, Package_LGA:Bosch_LGA-8_2x2.5mm_P0.65mm_ClockwisePinNumbering, symbol Sensor_Pressure:BMP280
- added U5: LIS2MDL, Package_LGA:LGA-12_2x2mm_P0.5mm, symbol Sensor_Magnetic:LIS2MDL
- added Y1: LFXTAL020423, LFXTAL020423:WE-XTAL_HC49_4HSMX, symbol 8mhz crystal:LFXTAL020423
- added Y2: ABMM2-32.768MHZ-E2F-T, ABMM2, symbol 32mhz crystal:ABMM2-32.768MHZ-E2F-T
- C5: value 47uF -> 22pF; footprint Capacitor_SMD:C_1206_3216Metric_Pad1.33x1.80mm_HandSolder -> Capacitor_SMD:C_0603_1608Metric_Pad1.08x0.95mm_HandSolder
- C6: value 330pF -> 22pF
- C7: value 47uF -> 12pF; footprint Capacitor_SMD:C_1206_3216Metric_Pad1.33x1.80mm_HandSolder -> Capacitor_SMD:C_0603_1608Metric_Pad1.08x0.95mm_HandSolder
Connections:
- net +3.3V: no longer J1.2 (Pin_2)
- net +VDC: now also J1.2 (Pin_2); no longer C5.2
- net GND: now also C5.2, C6.2, Y2.1 (X1), Y2.3 (X2); no longer C5.1, C7.2
- net MISO: now also U2.22 (PA6)
- net MOSI: now also U2.23 (PA7)
- net SCK: now also U2.29 (PB10)
- removed net 6V: C6.1, C7.1, J6.1 (Pin_1)
- net D10 renamed PB0
- net PB0: now also U2.26 (PB0)
- net D5 renamed PB3
- net PB3: now also U2.55 (PB3)
- net D6 renamed PB2
- net PB2: now also U2.28 (PB2)
- net D9 renamed PB1
- net PB1: now also U2.27 (PB1)
- new net: C5.1, U2.5 (PH0), Y1.1
- new net: J13.A1 (GND), J13.A12 (GND), J13.B1 (GND), J13.B12 (GND)
- new net: J13.A4 (VBUS), J13.A9 (VBUS), J13.B4 (VBUS), J13.B9 (VBUS)
- new net: U2.18 (VSS), U2.63 (VSS)
- new net: C8.2, U2.3 (PC14)
- new net: C7.2, U2.4 (PC15)
- new net: C6.1, U2.6 (PH1), Y1.2
- new net: U5.6 (GND), U5.8 (GND)
- new net: C7.1, Y2.2 (GND_1)
- new net: C8.1, Y2.4 (GND_2)
- no-connect marks 7 -> 4
Other:
- note added: "VDC? if not >10"
- note added: "is this VDC IN?"
- note added: "keep CLOSE to MCU, short traces"
- moved on the sheet: J1, J11, J6, Q1, R7

Commit message: added zoe
Parts:
- removed J1: ESC, Connector_PinHeader_1.00mm:PinHeader_1x06_P1.00mm_Vertical, symbol Connector:Conn_01x06_Socket
- removed J10, J7, J8, J9: M2, MountingHole:MountingHole_2.2mm_M2, symbol Connector_Generic_MountingPin:Conn_01x01_MountingPin
- added C10: 2.2uF, Capacitor_SMD:C_0603_1608Metric_Pad1.08x0.95mm_HandSolder, symbol Device:C
- added C11: 100nf, Capacitor_SMD:C_0603_1608Metric_Pad1.08x0.95mm_HandSolder, symbol Device:C
- added C9: 0.1uF, Capacitor_SMD:C_0603_1608Metric_Pad1.08x0.95mm_HandSolder, symbol Device:C
- added J1: Conn_01x08_Socket, symbol Connector:Conn_01x08_Socket
- added U4: ZOE-M8Q, RF_GPS:ublox_ZOE_M8, symbol RF_GPS:ZOE-M8Q
Connections:
- net +3.3V: now also MT1.5 (VDDIO), MT1.8 (VDD), C10.1, C11.1, C9.2
- net +VDC: now also J1.7 (Pin_7)
- net GND: now also MT1.6 (GND), MT1.7 (RESV__2), C10.2, C11.2, C9.1, J1.8 (Pin_8)
- net PB0: now also J1.6 (Pin_6)
- net PB1: now also J1.5 (Pin_5)
- net PB2: now also J1.4 (Pin_4)
- net PB3: now also J1.3 (Pin_3)
- net PC3: now reaches U2.11 (PC3)
- net PC3: now also J1.1 (Pin_1)
- new net: U4.A1 (GND), U4.A3 (GND), U4.A5 (GND), U4.A7 (GND), U4.A8 (GND), U4.A9 (GND), U4.B9 (GND), U4.C7 (GND), U4.C9 (GND), U4.D6 (GND), U4.D9 (GND), U4.E7 (GND), U4.F7 (GND), U4.G3 (GND), U4.G6 (GND), U4.G7 (GND), U4.J3 (GND), U4.J9 (GND)
- new net: U4.J1 (VCC), U4.J2 (VCC)
- no-connect marks 4 -> 5
Other:
- moved on the sheet: MT1, S1

Commit message: added new gps:m10q
Parts:
- removed U4: ZOE-M8Q, RF_GPS:ublox_ZOE_M8, symbol RF_GPS:ZOE-M8Q
- added U4: SAM-M10Q-00B, SAM-M10Q-00B:XCVR_SAM-M10Q-00B, symbol m10q:SAM-M10Q-00B
Connections:
- net MISO: now also MT1.1 (AP_SDO/AP_AD0)
- net MOSI: now also MT1.14 (AP_SDA/AP_SDIO/AP_SDI)
- net SCK: now also MT1.13 (AP_SCL/AP_SCLK), U2.21 (PA5)
- net PB4: now reaches U2.56 (PB4)
Other:
- moved on the sheet: J13, U3, U5

Commit message: slight labeling updates
Connections:
- net PB4: now also MT1.12 (AP_CS)
Other:
- note added: "change"
- note added: "this is the old baro, we don't need it anymore"
- moved on the sheet: U5
Changed lines of the file:
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@@
 	(generator_version "9.0")
 	(paper "A3")
+	(text "this is the old baro, we don't need it anymore"
+		(exclude_from_sim no)
+		(at 369.316 163.83 0)
+		(effects
+			(font
+				(size 1.27 1.27)
+			)
+		)
+	)
 	(text "keep CLOSE to MCU, short traces"
 		(exclude_from_sim no)
@@
 		)
 	)
+	(text "change\n"
+		(exclude_from_sim no)
+		(at 357.886 231.648 0)
+		(effects
+			(font
+				(size 1.27 1.27)
+			)
+		)
+	)
 	(text "is this VDC IN?\n"
 		(exclude_from_sim no)
@@
 	(wire
 		(pts
+			(xy 209.55 222.25) (xy 214.63 222.25)
+		)
+		(stroke
+			(width 0)
+			(type default)
+		)
+	)
+	(wire
+		(pts
 			(xy 377.19 232.41) (xy 381 232.41)
 		)
@@
 	(symbol
 		(lib_id "Sensor_Magnetic:LIS2MDL")
-		(at 203.2 163.83 0)
+		(at 214.63 163.83 0)
 		(unit 1)
 		(exclude_from_sim no)
@@
 		(fields_autoplaced yes)
 		(property "Reference" "U5"
-			(at 205.3433 176.53 0)
+			(at 216.7733 176.53 0)
 			(effects
 				(font
@@
 		)
 		(property "Value" "LIS2MDL"
-			(at 205.3433 179.07 0)
+			(at 216.7733 179.07 0)
 			(effects
 				(font
@@
 		)
 		(property "Footprint" "Package_LGA:LGA-12_2x2mm_P0.5mm"
-			(at 233.68 171.45 0)
+			(at 245.11 171.45 0)
 			(effects
 				(font
@@
 		)
 		(property "Datasheet" "https://www.st.com/resource/en/datasheet/lis2mdl.pdf"
-			(at 241.3 173.99 0)
+			(at 252.73 173.99 0)
 			(effects
 				(font
@@
 		)
 		(property "Description" "Ultra-low-power, 3-axis digital output magnetometer, LGA-12"
-			(at 203.2 163.83 0)
+			(at 214.63 163.83 0)
 			(effects
 				(font

Commit message: removed bmp280 and added 390
Parts:
- removed C10: 2.2uF, Capacitor_SMD:C_0603_1608Metric_Pad1.08x0.95mm_HandSolder, symbol Device:C
- removed C11: 100nf, Capacitor_SMD:C_0603_1608Metric_Pad1.08x0.95mm_HandSolder, symbol Device:C
- removed C9: 0.1uF, Capacitor_SMD:C_0603_1608Metric_Pad1.08x0.95mm_HandSolder, symbol Device:C
- removed J1: Conn_01x08_Socket, symbol Connector:Conn_01x08_Socket
- removed U3: BMP280, Package_LGA:Bosch_LGA-8_2x2.5mm_P0.65mm_ClockwisePinNumbering, symbol Sensor_Pressure:BMP280
- removed U4: SAM-M10Q-00B, SAM-M10Q-00B:XCVR_SAM-M10Q-00B, symbol m10q:SAM-M10Q-00B
- added J1: ESC, Connector_PinHeader_1.00mm:PinHeader_1x06_P1.00mm_Vertical, symbol Connector:Conn_01x06_Socket
- added J10, J7, J8, J9: M2, MountingHole:MountingHole_2.2mm_M2, symbol Connector_Generic_MountingPin:Conn_01x01_MountingPin
- added U3: BMP390, 10LGA_2X2X0p75_BOS, symbol bmp390:BMP390
Connections:
- net +3.3V: no longer MT1.5 (VDDIO), MT1.8 (VDD)
- net +VDC: now also J1.2 (Pin_2)
- net GND: now also J1.1 (Pin_1); no longer MT1.6 (GND), MT1.7 (RESV__2)
- net MISO: no longer MT1.1 (AP_SDO/AP_AD0)
- net MOSI: no longer MT1.14 (AP_SDA/AP_SDIO/AP_SDI)
- net PB0: now also J1.6 (Pin_6)
- net PB1: now also J1.5 (Pin_5)
- net PB2: now also J1.4 (Pin_4)
- net PB3: now also J1.3 (Pin_3)
- net SCK: no longer MT1.13 (AP_SCL/AP_SCLK), U2.21 (PA5)
- net PB4: no longer names the net of MT1.12 (AP_CS)
- net PB4: no longer U2.56 (PB4)
- net PC3: no longer names the net of U2.11 (PC3)
- no-connect marks 5 -> 4
Other:
- note removed: "change"
- note removed: "this is the old baro, we don't need it anymore"
- moved on the sheet: J13, MT1, S1, U5

Commit message: added bmp390 and wired it for 4 wire spi
miso = 4
mosi = 5
int = PB4
CSB = pb5
SCK = sck(pb10)
Parts:
- added C10, C9: 100nF, Capacitor_SMD:C_0603_1608Metric_Pad1.08x0.95mm_HandSolder, symbol Device:C
Connections:
- net +3.3V: now also U3.1 (VDDIO), U3.10 (VDD), C10.1, C9.1
- net GND: now also U3.3 (VSS), U3.8 (VSS), U3.9 (VSS), C10.2, C9.2
- net MISO: now also U3.4 (SDI)
- net MOSI: now also U3.5 (SDO)
- net SCK: now also U3.2 (SCK)
- net PB4: now reaches U2.56 (PB4)
- net PB4: now also U3.7 (INT)
- net PB5: now reaches U2.57 (PB5)
- net PB5: now also U3.6 (CSB)
Other:
- note added: "SDI SDO"
- moved on the sheet: U3

Commit message: added sam10mq to new rev
Parts:
- added C11: 100nF, Capacitor_SMD:C_0603_1608Metric_Pad1.08x0.95mm_HandSolder, symbol Device:C
- added U4: SAM-M10Q-00B, SAM-M10Q-00B:XCVR_SAM-M10Q-00B, symbol 10mq:SAM-M10Q-00B
Connections:
- net GND: now also C11.1
- net SCK: now also U5.1 (SCL/SPC)
- net at U5.10 (Vdd_IO): now also U5.9 (Vdd), C11.2

Commit message: added wiring for lis2mdl
Parts:
- removed C1: 100nf, Capacitor_SMD:C_0603_1608Metric_Pad1.08x0.95mm_HandSolder, symbol Device:C
- removed U1: MS560702BA03-50, pressure:SON125P300X500X100-8N, symbol pressure:MS560702BA03-50
- added C12: 220nF, Capacitor_SMD:C_0603_1608Metric_Pad1.08x0.95mm_HandSolder, symbol Device:C
- added R5: 10k, Resistor_SMD:R_0603_1608Metric_Pad0.98x0.95mm_HandSolder, symbol Device:R
Connections:
- net SDA is gone; now on net SDA (I2C3): R1.2
- net +3.3V: now also R5.1
- net GND: now also U5.6 (GND), U5.8 (GND), C12.1
- net MOSI: now also U5.7 (DRDY)
- net SCK: no longer R2.1, U5.1 (SCL/SPC)
- net SDA (I2C3): now reaches U2.40 (PC9)
- net SDA (I2C3): now also U5.4 (SDA/SDI/SDO)
- net SCL (I2C3): now reaches U2.41 (PA8)
- net SCL (I2C3): now also R2.1, U5.1 (SCL/SPC)
- net PB6: now reaches U2.58 (PB6)
- net PB6: now also U5.3 (~{CS}), R5.2
- net at U5.5 (C1): now also C12.2
- no-connect marks 4 -> 3
Other:
- moved on the sheet: C10, C9, MT1, U3
